Commit message: map generated

File: src/my_robot/urdf/my_robot.xacro (robot description, xacro)
@@ -149,4 +149,11 @@
     <dynamics damping="1.0" friction="1.0"/>
   </joint>
+<link name="camera_rgbd_frame">
+</link>
+<joint name="camera_rgbd_joint" type="fixed">
+    <origin xyz="0 0 0" rpy="-1.5707 0 -1.5707"/>
+    <parent link="camera"/>
+    <child link="camera_rgbd_frame"/>
+  </joint>
 <link name='hokuyo'>
     <inertial>
